File: rev1/Top/first_keyboard.kicad_pcb (KiCad board)
At the start: 2 copper layers, 271.5 x 88.6 mm, 47 parts, among them SW1 SW_Push, SW10 SW_Push, SW11 SW_Push, SW12 SW_Push, SW13 SW_Push, SW14 SW_Push, SW15 SW_Push, SW16 SW_Push, SW17 SW_Push, SW18 SW_Push, SW19 SW_Push, SW2 SW_Push, SW20 SW_Push, SW21 SW_Push, SW22 SW_Push, SW23 SW_Push, SW24 SW_Push, SW25 SW_Push, SW26 SW_Push, SW27 SW_Push, SW28 SW_Push, SW29 SW_Push, SW3 SW_Push, SW30 SW_Push, SW31 SW_Push, SW32 SW_Push, SW33 SW_Push, SW34 SW_Push, SW35 SW_Push, SW36 SW_Push, SW37 SW_Push, SW38 SW_Push, SW39 SW_Push, SW4 SW_Push, SW5 SW_Push, SW6 SW_Push, SW7 SW_Push, SW8 SW_Push, SW9 SW_Push

Commit message: add: top_plate
Parts:
- removed REF** (x8): MountingHole_3.2mm_M3, MountingHole:MountingHole_3.2mm_M3
- added Ref1: Val**, MountingHole:MountingHole_3.2mm_M3, F.Cu at (47.6, 100.0)
- added Ref2: Val**, MountingHole:MountingHole_3.2mm_M3, F.Cu at (364.3, 100.0)
- added Ref3: Val**, MountingHole:MountingHole_3.2mm_M3, F.Cu at (171.4, 114.3)
- added Ref4: Val**, MountingHole:MountingHole_3.2mm_M3, F.Cu at (240.5, 114.3)
- added Ref5: Val**, MountingHole:MountingHole_3.2mm_M3, F.Cu at (102.4, 173.8)
- added Ref6: Val**, MountingHole:MountingHole_3.2mm_M3, F.Cu at (309.6, 173.8)
- added SW40: SW_Push, kbd_SW_Hole:SW_Hole_1u, F.Cu at (356.9, 115.8)
- added SW41: SW_Push, kbd_SW_Hole:SW_Hole_2u, F.Cu at (356.9, 144.4)
- SW39: footprint kbd_SW_Hole:SW_Hole_2u -> kbd_SW_Hole:SW_Hole_1u
- moved SW22 146.2 mm to (261.6, 115.8)
- moved SW13 137.1 mm to (130.8, 173.0)
- moved SW17 137.1 mm to (149.8, 173.0)
- moved SW29 136.2 mm to (261.6, 173.0)
- moved SW32 127.4 mm to (299.7, 153.9)
- moved SW23 123.8 mm to (261.6, 134.9)
- moved SW24 123.8 mm to (261.6, 153.9)
- moved SW21 119.6 mm to (168.9, 173.0)
- moved SW33 118.5 mm to (280.7, 173.0)
- moved SW20 113.0 mm to (149.8, 153.9)
- moved SW9 113.0 mm to (92.7, 153.9)
- moved SW25 111.5 mm to (242.6, 173.0)
- moved SW35 111.5 mm to (318.8, 134.9)
- moved SW36 111.5 mm to (318.8, 153.9)
- moved SW38 111.5 mm to (337.8, 134.9)
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Other:
- board size 271.5 x 88.6 mm -> 331 x 95.2 mm

Commit message: feat: 刻印追加
Other:
- board text added: "madbd v0.0.2 Design by: @amkkr X: @ama_O255"
Changed lines of the file:
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@@
   (gr_line (start 290.5125 188.11875) (end 121.44375 188.11875)
     (stroke (width 0.2) (type default)) (layer "Edge.Cuts"))
+  (gr_text "madbd v0.0.2	Design by: @amkkr\n						X: @ama_O255" (at 319.0875 166.6875) (layer "F.SilkS" knockout)
+    (effects (font (size 1.5 1.5) (thickness 0.1875)))
+  )
 )
