File: rev1/Top/first_keyboard.kicad_pcb (KiCad board)
At the start: 2 copper layers, 331 x 95.2 mm, 47 parts, among them SW1 SW_Push, SW10 SW_Push, SW11 SW_Push, SW12 SW_Push, SW13 SW_Push, SW14 SW_Push, SW15 SW_Push, SW16 SW_Push, SW17 SW_Push, SW18 SW_Push, SW19 SW_Push, SW2 SW_Push, SW20 SW_Push, SW21 SW_Push, SW22 SW_Push, SW23 SW_Push, SW24 SW_Push, SW25 SW_Push, SW26 SW_Push, SW27 SW_Push, SW28 SW_Push, SW29 SW_Push, SW3 SW_Push, SW30 SW_Push, SW31 SW_Push, SW32 SW_Push, SW33 SW_Push, SW34 SW_Push, SW35 SW_Push, SW36 SW_Push, SW37 SW_Push, SW38 SW_Push, SW39 SW_Push, SW4 SW_Push, SW40 SW_Push, SW41 SW_Push, SW5 SW_Push, SW6 SW_Push, SW7 SW_Push, SW8 SW_Push, SW9 SW_Push

Commit message: feat: 輪郭線変更
Parts:
- removed Ref1, Ref2, Ref3, Ref4, Ref5, Ref6: Val**, MountingHole:MountingHole_3.2mm_M3
- added D1: D, kbd_Parts:Diode_TH_SMD, F.Cu at (85.7, 134.3)
- added D10: D, kbd_Parts:Diode_TH_SMD, F.Cu at (142.9, 129.5)
- added D11: D, kbd_Parts:Diode_TH_SMD, F.Cu at (142.9, 148.6)
- added D12: D, kbd_Parts:Diode_TH_SMD, F.Cu at (142.9, 167.6)
- added D13: D, kbd_Parts:Diode_TH_SMD, F.Cu at (161.9, 186.7)
- added D14: D, kbd_Parts:Diode_TH_SMD, F.Cu at (161.9, 129.5)
- added D15: D, kbd_Parts:Diode_TH_SMD, F.Cu at (161.9, 148.6)
- added D16: D, kbd_Parts:Diode_TH_SMD, F.Cu at (161.9, 167.6)
- added D17: D, kbd_Parts:Diode_TH_SMD, F.Cu at (181.0, 191.5)
- added D18: D, kbd_Parts:Diode_TH_SMD, F.Cu at (181.0, 134.3)
- added D19: D, kbd_Parts:Diode_TH_SMD, F.Cu at (181.0, 153.4)
- added D2: D, kbd_Parts:Diode_TH_SMD, F.Cu at (85.7, 153.4)
- added D20: D, kbd_Parts:Diode_TH_SMD, F.Cu at (181.0, 172.4)
- added D21: D, kbd_Parts:Diode_TH_SMD, F.Cu at (200.0, 193.8)
- added D22: D, kbd_Parts:Diode_TH_SMD, F.Cu at (266.7, 134.3)
- added D23: D, kbd_Parts:Diode_TH_SMD, F.Cu at (266.7, 153.4)
- added D24: D, kbd_Parts:Diode_TH_SMD, F.Cu at (266.7, 172.4)
- added D25: D, kbd_Parts:Diode_TH_SMD, F.Cu at (247.7, 193.8)
- added D26: D, kbd_Parts:Diode_TH_SMD, F.Cu at (285.8, 129.5)
- added D27: D, kbd_Parts:Diode_TH_SMD, F.Cu at (285.8, 148.6)
- added D28: D, kbd_Parts:Diode_TH_SMD, F.Cu at (285.8, 167.6)
- added D29: D, kbd_Parts:Diode_TH_SMD, F.Cu at (266.7, 191.5)
- added D3: D, kbd_Parts:Diode_TH_SMD, F.Cu at (85.7, 172.4)
- added D30: D, kbd_Parts:Diode_TH_SMD, F.Cu at (285.8, 186.7)
- added D31: D, kbd_Parts:Diode_TH_SMD, F.Cu at (304.8, 129.5)
- added D32: D, kbd_Parts:Diode_TH_SMD, F.Cu at (304.8, 148.6)
- added D33: D, kbd_Parts:Diode_TH_SMD, F.Cu at (304.8, 167.6)
- added D34: D, kbd_Parts:Diode_TH_SMD, F.Cu at (323.9, 129.5)
- added D35: D, kbd_Parts:Diode_TH_SMD, F.Cu at (323.9, 148.6)
- added D36: D, kbd_Parts:Diode_TH_SMD, F.Cu at (323.9, 167.6)
- added D37: D, kbd_Parts:Diode_TH_SMD, F.Cu at (342.9, 129.5)
- added D38: D, kbd_Parts:Diode_TH_SMD, F.Cu at (342.9, 148.6)
- added D39: D, kbd_Parts:Diode_TH_SMD, F.Cu at (342.9, 167.6)
- added D4: D, kbd_Parts:Diode_TH_SMD, F.Cu at (104.8, 129.5)
- added D40: D, kbd_Parts:Diode_TH_SMD, F.Cu at (361.9, 134.3)
- added D41: D, kbd_Parts:Diode_TH_SMD, F.Cu at (357.2, 167.6)
- added D5: D, kbd_Parts:Diode_TH_SMD, F.Cu at (104.8, 148.6)
- added D6: D, kbd_Parts:Diode_TH_SMD, F.Cu at (104.8, 167.6)
- added D7: D, kbd_Parts:Diode_TH_SMD, F.Cu at (123.8, 129.5)
- added D8: D, kbd_Parts:Diode_TH_SMD, F.Cu at (123.8, 148.6)
- added D9: D, kbd_Parts:Diode_TH_SMD, F.Cu at (123.8, 167.6)
- added U1: Pico, RPi_Pico:RPi_Pico_SMD_TH, F.Cu at (216.7, 138.1)
- SW1, SW10, SW11, SW12, SW13, SW14, SW15, SW16, SW17, SW18, SW19, SW2, SW20, SW21, SW22, SW23, SW24, SW25, SW26, SW27, SW28, SW29, SW3, SW30, SW31, SW32, SW33, SW34, SW35, SW36, SW37, SW38, SW39, SW4, SW40, SW5, SW6, SW7, SW8, SW9: footprint kbd_SW_Hole:SW_Hole_1u -> kbd_SW:CherryMX_Hotswap_1u
- SW41: footprint kbd_SW_Hole:SW_Hole_2u -> kbd_SW:CherryMX_Hotswap_2u
- moved SW30 68.5 mm to (278.6, 181.0)
- moved SW21 28.4 mm to (192.9, 188.1)
- moved SW17 27.2 mm to (173.8, 185.7)
- moved SW18 27.2 mm to (173.8, 128.6)
- moved SW19 27.2 mm to (173.8, 147.6)
- moved SW20 27.2 mm to (173.8, 166.7)
- moved SW1 27.2 mm to (78.6, 128.6)
- moved SW2 27.2 mm to (78.6, 147.6)
- moved SW3 27.2 mm to (78.6, 166.7)
- moved SW13 25.3 mm to (154.8, 181.0)
- moved SW14 25.3 mm to (154.8, 123.8)
- moved SW15 25.3 mm to (154.8, 142.9)
- moved SW16 25.3 mm to (154.8, 161.9)
- moved SW7 25.3 mm to (116.7, 123.8)
- moved SW8 25.3 mm to (116.7, 142.9)
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Other:
- board size 331 x 95.2 mm -> 300 x 88.1 mm
- board text removed: "madbd v0.0.2 Design by: @amkkr X: @ama_O255"

Commit message: feat: スペース繋げて外形変更
Parts:
- added Ref**: Val**, kbd_Hole:m2_Screw_Hole, F.Cu at (86.5, 118.0)
- added Ref**: Val**, kbd_Hole:m2_Screw_Hole, F.Cu at (346.5, 118.0)
- SW1, SW10, SW11, SW12, SW13, SW14, SW15, SW16, SW17, SW18, SW19, SW2, SW20, SW21, SW22, SW23, SW24, SW25, SW26, SW27, SW28, SW29, SW3, SW30, SW31, SW32, SW33, SW34, SW35, SW36, SW37, SW38, SW39, SW4, SW40, SW5, SW6, SW7, SW8, SW9: footprint kbd_SW:CherryMX_Hotswap_1u -> kbd_SW_Hole:SW_Hole_TH_1u
- SW41: footprint kbd_SW:CherryMX_Hotswap_2u -> kbd_SW_Hole:SW_Hole_TH_2u
Other:
- outline, holes or cut-outs redrawn

Commit message: feat: Topからダイオード削除
Parts:
- removed D1, D10, D11, D12, D13, D14, D15, D16, D17, D18, D19, D2, D20, D21, D22, D23, D24, D25, D26, D27, D28, D29, D3, D30, D31, D32, D33, D34, D35, D36, D37, D38, D39, D4, D40, D41, D5, D6, D7, D8, D9: D, kbd_Parts:Diode_TH_SMD
- removed Ref** (x2): Val**, kbd_Hole:m2_Screw_Hole
- moved SW37 28.6 mm to (307.2, 123.8)
- moved SW38 28.6 mm to (307.2, 142.9)
- moved SW39 28.6 mm to (307.2, 161.9)
- moved SW22 28.6 mm to (231.0, 128.6)
- moved SW23 28.6 mm to (231.0, 147.6)
- moved SW24 28.6 mm to (231.0, 166.7)
- moved SW25 28.6 mm to (211.9, 188.1)
- moved SW26 28.6 mm to (250.0, 123.8)
- moved SW27 28.6 mm to (250.0, 142.9)
- moved SW28 28.6 mm to (250.0, 161.9)
- moved SW29 28.6 mm to (231.0, 185.7)
- moved SW30 28.6 mm to (250.0, 181.0)
- moved SW31 28.6 mm to (269.1, 123.8)
- moved SW32 28.6 mm to (269.1, 142.9)
- moved SW33 28.6 mm to (269.1, 161.9)
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Other:
- board size 300 x 88.1 mm -> 271.5 x 88.1 mm

Commit message: feat: Topネジ穴追加
Parts:
- removed U1: Pico, RPi_Pico:RPi_Pico_SMD_TH
- added Ref**: Val**, kbd_Hole:m2_Screw_Hole, F.Cu at (86.5, 117.0)
- added Ref**: Val**, kbd_Hole:m2_Screw_Hole, F.Cu at (314.5, 173.0)
- added Ref**: Val**, kbd_Hole:m2_Screw_Hole, F.Cu at (162.5, 192.0)
- added Ref**: Val**, kbd_Hole:m2_Screw_Hole, F.Cu at (318.5, 117.0)
- added Ref**: Val**, kbd_Hole:m2_Screw_Hole, F.Cu at (143.5, 173.0)
- added Ref**: Val**, kbd_Hole:m2_Screw_Hole, F.Cu at (238.5, 117.0)
- added Ref**: Val**, kbd_Hole:m2_Screw_Hole, F.Cu at (90.5, 173.0)
- added Ref**: Val**, kbd_Hole:m2_Screw_Hole, F.Cu at (242.5, 192.0)
- added Ref**: Val**, kbd_Hole:m2_Screw_Hole, F.Cu at (261.5, 173.0)
- added Ref**: Val**, kbd_Hole:m2_Screw_Hole, F.Cu at (166.5, 117.0)
Other:
- outline, holes or cut-outs redrawn

Commit message: feat: ６角スペーサー穴追加
Parts:
- removed the Ref** at (143.5, 173.0)
- removed the Ref** at (261.5, 173.0)

Commit message: feat: TOPに模様追加
Routing:
- added copper zone on B.Cu, net (none)
- added copper zone on F.Cu, net (none)

Commit message: feat: ドリルファイル生成
Parts:
- SW1, SW10, SW11, SW12, SW13, SW14, SW15, SW16, SW17, SW18, SW19, SW2, SW20, SW21, SW22, SW23, SW24, SW25, SW26, SW27, SW28, SW29, SW3, SW30, SW31, SW32, SW33, SW34, SW35, SW36, SW37, SW38, SW39, SW4, SW40, SW5, SW6, SW7, SW8, SW9: footprint kbd_SW_Hole:SW_Hole_TH_1u -> kbd_SW_Hole:SW_Hole_1u
- SW41: footprint kbd_SW_Hole:SW_Hole_TH_2u -> kbd_SW_Hole:SW_Hole_2u
