File: rev1/Top/first_keyboard_top.kicad_pcb (KiCad board)
At the start: 2 copper layers, 352.4 x 109.5 mm, 80 parts, among them SW1 SW_Push, SW10 SW_Push, SW11 SW_Push, SW12 SW_Push, SW13 SW_Push, SW14 SW_Push, SW15 SW_Push, SW16 SW_Push, SW17 SW_Push, SW18 SW_Push, SW19 SW_Push, SW2 SW_Push, SW20 SW_Push, SW21 SW_Push, SW22 SW_Push, SW23 SW_Push, SW24 SW_Push, SW25 SW_Push, SW26 SW_Push, SW27 SW_Push, SW28 SW_Push, SW29 SW_Push, SW3 SW_Push, SW30 SW_Push, SW31 SW_Push, SW32 SW_Push, SW33 SW_Push, SW34 SW_Push, SW35 SW_Push, SW36 SW_Push, SW37 SW_Push, SW38 SW_Push, SW39 SW_Push, SW4 SW_Push, SW40 SW_Push, SW41 SW_Push, SW42 SW_Push, SW43 SW_Push, SW44 SW_Push, SW45 SW_Push, SW46 SW_Push, SW47 SW_Push, SW48 SW_Push, SW49 SW_Push, SW5 SW_Push, SW50 SW_Push, SW51 SW_Push, SW52 SW_Push, SW53 SW_Push, SW54 SW_Push, SW55 SW_Push, SW56 SW_Push, SW57 SW_Push, SW58 SW_Push, SW59 SW_Push, SW6 SW_Push, SW60 SW_Push, SW7 SW_Push, SW8 SW_Push, SW9 SW_Push

Commit message: feat: ネジ穴位置調整
Parts:
- removed Ref** (x20): Val**, kbd_Hole:m2_Screw_Hole
- added ref: val, kbd_Hole:m2_Screw_Hole, F.Cu at (40.2, 52.7)
- added ref: val, kbd_Hole:m2_Screw_Hole, F.Cu at (288.8, 73.0)
- added ref: val, kbd_Hole:m2_Screw_Hole, F.Cu at (277.3, 154.3)
- added ref: val, kbd_Hole:m2_Screw_Hole, F.Cu at (230.7, 154.3)
- added ref: val, kbd_Hole:m2_Screw_Hole, F.Cu at (368.8, 76.8)
- added ref: val, kbd_Hole:m2_Screw_Hole, F.Cu at (344.6, 131.4)
- added ref: val, kbd_Hole:m2_Screw_Hole, F.Cu at (219.2, 73.0)
- added ref: val, kbd_Hole:m2_Screw_Hole, F.Cu at (40.2, 146.7)
- added ref: val, kbd_Hole:m2_Screw_Hole, F.Cu at (157.0, 75.6)
- added ref: val, kbd_Hole:m2_Screw_Hole, F.Cu at (117.6, 131.4)
- added ref: val, kbd_Hole:m2_Screw_Hole, F.Cu at (115.1, 52.7)
- added ref: val, kbd_Hole:m2_Screw_Hole, F.Cu at (163.4, 131.4)
- moved SW15 0.95 mm to (358.6, 85.7)
- moved SW31 0.95 mm to (358.6, 104.8)
- moved SW47 0.95 mm to (358.6, 123.8)
- moved SW55 0.95 mm to (263.4, 147.6)
- moved SW22 0.95 mm to (149.1, 104.8)
- moved SW24 0.95 mm to (187.2, 100.0)
- moved SW38 0.95 mm to (149.1, 123.8)
- moved SW40 0.95 mm to (187.2, 119.1)
- moved SW54 0.95 mm to (244.3, 147.6)
- moved SW6 0.95 mm to (149.1, 85.7)
- moved SW8 0.95 mm to (187.2, 81.0)
- moved SW1 0.95 mm to (49.1, 61.9)
- moved SW17 0.95 mm to (49.1, 81.0)
- moved SW18 0.95 mm to (68.1, 81.0)
- moved SW19 0.95 mm to (87.2, 81.0)
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
Commit message: add: fox
Parts:
- added G***: LOGO, Top:fox, F.Cu at (252.4, 107.2)
