File: rev1/first_keyboard.kicad_pcb (KiCad board)
At the start: 2 copper layers, 331 x 95.2 mm, 90 parts, among them SW1 SW_Push, SW10 SW_Push, SW11 SW_Push, SW12 SW_Push, SW13 SW_Push, SW14 SW_Push, SW15 SW_Push, SW16 SW_Push, SW17 SW_Push, SW18 SW_Push, SW19 SW_Push, SW2 SW_Push, SW20 SW_Push, SW21 SW_Push, SW22 SW_Push, SW23 SW_Push, SW24 SW_Push, SW25 SW_Push, SW26 SW_Push, SW27 SW_Push, SW28 SW_Push, SW29 SW_Push, SW3 SW_Push, SW30 SW_Push, SW31 SW_Push, SW32 SW_Push, SW33 SW_Push, SW34 SW_Push, SW35 SW_Push, SW36 SW_Push, SW37 SW_Push, SW38 SW_Push, SW39 SW_Push, SW4 SW_Push, SW40 SW_Push, SW41 SW_Push, SW42 SW_Push, SW5 SW_Push, SW6 SW_Push, SW7 SW_Push, SW8 SW_Push, SW9 SW_Push, U1 Pico

Commit message: feat: PCBの配置を変更
Parts:
- removed Ref1, Ref2, Ref3, Ref4, Ref5, Ref6: Val**, kbd_Hole:m3_Spacer_Hole
- removed SW42: SW_Push, kbd_Parts:ResetSW
- D1, D10, D11, D12, D13, D14, D15, D16, D17, D18, D19, D2, D20, D21, D22, D23, D24, D25, D26, D27, D28, D29, D3, D30, D31, D32, D33, D34, D35, D36, D37, D38, D39, D4, D40, D41, D5, D6, D7, D8, D9, U1: moved to F.Cu
- moved D39 43.3 mm to (371.5, 164.3)
- moved D41 43.2 mm to (383.4, 164.3)
- moved D22 36.2 mm to (288.1, 126.2)
- moved D23 36.2 mm to (288.1, 145.3)
- moved D24 36.2 mm to (288.1, 164.3)
- moved D25 36.2 mm to (269.1, 183.4)
- moved D29 36.2 mm to (288.1, 183.4)
- moved D26 36.2 mm to (307.2, 126.2)
- moved D27 36.2 mm to (307.2, 145.3)
- moved D28 36.2 mm to (307.2, 164.3)
- moved D30 36.2 mm to (326.2, 126.2)
- moved D31 36.2 mm to (326.2, 145.3)
- moved D32 36.2 mm to (326.2, 164.3)
- moved D33 36.2 mm to (307.2, 183.4)
- moved D34 36.2 mm to (345.3, 126.2)
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Connections:
- U1 pad 10: Col10 -> Row1
- U1 pad 11: Col9 -> Row2
- U1 pad 12: Col8 -> Row3
- U1 pad 14: Col7 -> Col0
- U1 pad 15: Col6 -> Col1
- U1 pad 16: Col5 -> Col2
- U1 pad 17: Col4 -> Col3
- U1 pad 19: Col3 -> Col4
- U1 pad 20: Col2 -> Col5
- U1 pad 21: Col1 -> Col11
- U1 pad 22: Col0 -> Col10
- U1 pad 24: Row3 -> Col9
- U1 pad 25: Row2 -> Col8
- U1 pad 26: Row1 -> Col7
- U1 pad 27: Row0 -> Col6
- U1 pad 30: reset -> unconnected-(U1-RUN-Pad30)
- U1 pad 40: Net-(U1-VBUS) -> GND
- U1 pad 9: Col11 -> Row0
Routing:
- net Row0: track 367.8 -> 0.00 mm
- net Row1: track 338.1 -> 0.00 mm, vias 1 -> 0
- net Row2: track 325.3 -> 0.00 mm, vias 2 -> 0
- net Row3: track 210.3 -> 0.00 mm
- net Col0: track 199.0 -> 0.00 mm, vias 1 -> 0
- net Col2: track 195.1 -> 0.00 mm, vias 1 -> 0
- net Col3: track 182.2 -> 0.00 mm, vias 1 -> 0
- net Col1: track 180.4 -> 0.00 mm, vias 1 -> 0
- net Col4: track 165.8 -> 0.00 mm, vias 2 -> 0
- net Col11: track 165.5 -> 0.00 mm, vias 1 -> 0
- net Col10: track 159.7 -> 0.00 mm, vias 1 -> 0
- net Col8: track 153.5 -> 0.00 mm, vias 1 -> 0
- net Col5: track 148.1 -> 0.00 mm, vias 2 -> 0
- net Col9: track 140.4 -> 0.00 mm, vias 1 -> 0
- net Col7: track 122.1 -> 0.00 mm
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Other:
- board outline removed

Commit message: fix: 左右とpicoの整列
Parts:
- moved U1 4.39 mm to (207.5, 133.3)
Changed lines of the file:
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@@
   )
   (footprint "RPi_Pico:RPi_Pico_SMD_TH" (layer "F.Cu")
-    (at 211.93125 133.35)
+    (at 207.54375 133.35)
     (descr "Through hole straight pin header, 2x20, 2.54mm pitch, double rows")
     (tags "Through hole pin header THT 2x20 2.54mm double row")
@@
       (net 74 "unconnected-(U1-SWDIO-Pad43)") (pinfunction "SWDIO") (pintype "bidirectional+no_connect"))
   )
+  (group "" (id 0ac3a1c4-a834-431d-881a-eefc23ac47ea)
+    (members
+      012d0bbc-c991-48b7-a9c3-a4bf0702b85b
+      019946a3-0451-45be-bb2a-9411ba8dfa54
+      063f3ef4-d551-4894-a1a5-a3b7b1e9be3a
+      1486658f-b713-4c7c-837c-d00a88680b5c
+      1d9651bf-7796-45ea-8bfe-e4a6342e1f34
+      24d4b9b0-eb60-4809-b540-9031c6aa4572
+      2552e0f4-a58c-4955-abc7-6eda5e731ad0
+      2c70b89e-101d-4395-b57a-f2897b5730e2
+      2e742a16-e774-4dd4-a9e7-bd98bc12e477
+      2f03d40c-de77-40a1-a33a-fd2395aefff9
+      2f416950-f953-4939-82c5-5a8ace22185b
+      312a4c69-7f8a-43b8-86e2-b6eb86d0f5ce
+      580411b8-5f50-4bef-b092-95539251e80e
+      5c5715c8-42c5-4ac2-a07c-5ab38c5028e7
+      5f60d736-09fb-4908-b4e5-b62b6537817b
+      60245ab0-c055-4749-a8b9-e506b5842b97
+      6471bc29-87de-49d4-a200-9cf835def8c5
+      73650dbf-5b15-4747-8e36-4f242b3b82e8
+      78345dea-3273-413c-a2a6-f94e9696e15e
+      8bb0c742-d3d6-472a-a46a-6fa19350f769
+      9370ebb2-2ae3-4827-b4e4-49341229cae2
+      962c4abd-2cf1-4ea0-8859-9adb3e95705d
+      9a7cbe31-a63b-4270-a824-693055ff881f
+      9b075ca8-e758-441b-8914-4e13b45d4eef
+      9d662371-fb2f-43af-9ce8-de5cfe563da1
+      a7c69859-9bd5-41b9-8ed0-075a2dddb52c
+      a84ca691-0233-42d4-aac2-f7a9c0490f6d
+      a8e650b7-5022-4bf1-9af8-1af162efa941
+      abc220ad-3e44-4ab4-b6b6-84f4176312ed
+      aff8297f-1f57-4fbb-af0d-b1b3d7198748
+      b2a287ee-2d96-43a4-8e02-c3177d15dee5
+      b7425290-8e62-4ea3-a185-9aa1a39f97b7
+      bb12a942-ca70-4052-b3a6-ffb7a1735ca4
+      be93b58d-10c1-47f1-a928-2cf1ee23f56e
+      c50f161f-66cd-43ac-829a-28669af9b65f
+      d49bfea6-3068-4a84-aace-ff23860e199a
+      e0339819-ca7c-4aa8-bec9-c3869ae452c3
+      e11d23ee-3482-4ebe-b562-c255197ea5fd
+      eae43429-e45c-4b62-a999-391ddc07b657
+      ee3691ea-5ead-4951-bf0c-1527559c45c8
+    )
+  )
+  (group "" (id af2218d8-2dd4-47ac-8b53-74f56c7c5f5c)
+    (members
+      082319f0-3429-419a-8e27-fc1732ba7365
+      18168899-0915-4371-9ae7-6525f5697281
+      1cf0fe2a-55e7-40d5-95ee-7cf8e9b545e9
+      1d263154-1689-4456-925b-7400b34d2285
+      255f3cdc-3eab-4952-8c70-01cdce16be26
+      2a117461-4fa8-4367-87e7-5596f5c06cbe
+      2e33eed3-31b3-4159-b25e-f764429bb112
+      3af0f068-d567-41b4-8305-56c01be11c99
+      3bc6e94e-d3a3-434c-8c5d-359b43de264f
+      3c772cf1-4b43-4d9e-aadc-3b649a1be07a
+      40698693-5d86-47ec-88e8-ef66e18c6951
+      41098754-2ae1-44be-8953-7d3d3d0105fe
+      463d3815-9677-4f7a-90f0-91940ca64131
+      5318bd59-d895-4fd2-a3c1-1a69b7a5a89c
+      5b45a620-c828-4e46-8a7a-1a320789905e
+      6ab9c5b8-5f8c-4ac3-b26c-7e3ea6bd4982
+      6d1d916e-f84e-4972-b1ca-bd03356acb6c
+      72c09cf5-95ce-4cf0-99bb-8b1ff452d7a4
+      8f352e6d-94bd-45e5-a250-f1e97f33fffb
+      96367ea9-320c-4485-a46d-04aef7731424
+      a497f8d4-bfe2-4924-ad20-dce76f592652
+      ad30e082-b409-48d5-9cb3-a2faae83d234
+      adf27df8-a312-48f1-9fe3-62a17b3a24a0
+      b6b19121-8033-4256-a0c2-1d2a23ac7301
+      bd8e4896-be16-4051-a5b9-97a8941ee0c5
+      bff5201c-d15f-4fb3-a461-d37ccd8c58cb
+      c737adbb-9deb-4225-8852-4cfd3ae9b98a
+      ce9d699d-2619-457c-8801-310ce87bf7f8
+      cf089b7a-ce34-499f-ae79-2b655d7a3469
+      d0116e12-7ed0-4bf3-9646-938da9fbf5c6
+      d7cdd4cf-c6ff-45f7-8c74-104ae23522b0
+      d801a585-27f1-4d3b-a974-4be7fc7d3d07
+      e175d532-cf80-4e1b-9108-53eabef245f0
+      e236cccb-6224-479d-803c-9e52daead8d8
+      e278fcda-7012-4fd9-b596-e54aa62904dd
+      e28bafb1-a35a-426c-b3ca-97ce2a99101f
+      e805f016-c64e-4a35-bc92-f1e98730882f
+      e81c2720-f355-46c4-82ed-6b90991b000f
+      eba44a67-a337-4b4f-b48a-71cd132ef261
+      ebd1fd8c-0b8b-4b5d-a35a-b1322f201a63
+      ef421a21-5c48-4afe-b82e-6dbbd028d395
+      f115dcdf-9698-4c38-8aee-a55efa1edbde
+    )
+  )
 )

Commit message: feat: 角度8, 左右幅初期位置
Parts:
- moved U1 11.9 mm to (207.2, 145.3)
- moved D21 10.4 mm to (159.0, 192.3), turned to 82 degrees
- moved D40 9.92 mm to (379.4, 117.1), turned to 98 degrees
- moved D41 9.57 mm to (384.7, 154.8), turned to 98 degrees
- moved SW1 8.96 mm to (45.0, 113.7), turned to -8 degrees
- moved SW40 8.96 mm to (369.3, 113.7), turned to 8 degrees
- moved SW25 8.87 mm to (264.1, 186.2), turned to 8 degrees
- moved SW21 8.87 mm to (150.3, 186.2), turned to -8 degrees
- moved SW2 8.13 mm to (42.4, 132.6), turned to -8 degrees
- moved SW3 8.13 mm to (39.7, 151.4), turned to -8 degrees
- moved D25 8.07 mm to (274.2, 189.6), turned to 98 degrees
- moved D17 8.07 mm to (140.2, 189.6), turned to 82 degrees
- moved SW41 8.02 mm to (373.3, 142.0), turned to -82 degrees
- moved D39 7.95 mm to (372.9, 156.5), turned to 98 degrees
- moved D1 7.48 mm to (53.8, 119.8), turned to 82 degrees
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
Commit message: feat: lotate 12, width 4
Parts:
- moved SW40 41.7 mm to (328.2, 106.9), turned to 12 degrees
- moved D40 41.6 mm to (338.5, 109.6), turned to 102 degrees
- moved SW37 41.3 mm to (309.5, 110.9), turned to 12 degrees
- moved D37 41.2 mm to (319.8, 113.5), turned to 102 degrees
- moved SW34 40.9 mm to (290.9, 114.8), turned to 12 degrees
- moved D34 40.8 mm to (301.2, 117.5), turned to 102 degrees
- moved SW30 40.6 mm to (272.3, 118.8), turned to 12 degrees
- moved D30 40.4 mm to (282.6, 121.5), turned to 102 degrees
- moved SW26 40.3 mm to (253.6, 122.8), turned to 12 degrees
- moved D26 40.1 mm to (263.9, 125.4), turned to 102 degrees
- moved SW38 40.0 mm to (313.5, 129.5), turned to 12 degrees
- moved SW22 40.0 mm to (235.0, 126.7), turned to 12 degrees
- moved D38 39.9 mm to (323.8, 132.2), turned to 102 degrees
- moved SW41 39.8 mm to (334.1, 134.9), turned to -78 degrees
- moved D22 39.8 mm to (245.3, 129.4), turned to 102 degrees
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
Commit message: feat: lotate 10 両端のキーは無回転
Parts:
- moved D40 23.6 mm to (352.4, 128.6), turned to 90 degrees
- moved SW1 22.4 mm to (61.9, 123.8), turned to 0 degrees
- moved SW40 22.4 mm to (342.9, 123.8), turned to 0 degrees
- moved D41 20.7 mm to (352.4, 166.7), turned to 90 degrees
- moved SW2 20.4 mm to (61.9, 142.9), turned to 0 degrees
- moved D1 20.2 mm to (71.4, 128.6), turned to 90 degrees
- moved SW41 19.6 mm to (342.9, 152.4), turned to -90 degrees
- moved SW3 19.0 mm to (61.9, 161.9), turned to 0 degrees
- moved D2 18.2 mm to (71.4, 147.6), turned to 90 degrees
- moved D3 16.8 mm to (71.4, 166.7), turned to 90 degrees
- moved D39 6.94 mm to (327.8, 150.0), turned to 100 degrees
- moved D21 4.89 mm to (186.5, 188.6), turned to 80 degrees
- moved SW21 4.54 mm to (178.0, 182.3), turned to -10 degrees
- moved SW25 4.44 mm to (226.8, 182.4), turned to 10 degrees
- moved D18 4.35 mm to (177.7, 129.0), turned to 80 degrees
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
Commit message: feat: 小指カラムをさげる part1
Parts:
- moved D37 26.8 mm to (327.1, 138.7), turned to -177 degrees
- moved D39 26.7 mm to (329.1, 176.7), turned to -177 degrees
- moved D38 26.7 mm to (328.1, 157.7), turned to -177 degrees
- moved SW37 25.3 mm to (326.6, 129.2), turned to 3 degrees
- moved SW38 24.1 mm to (327.6, 148.2), turned to 3 degrees
- moved SW6 23.8 mm to (100.0, 167.2), turned to -3 degrees
- moved D6 23.6 mm to (99.5, 176.7), turned to 177 degrees
- moved D5 23.1 mm to (100.5, 157.6), turned to 177 degrees
- moved SW39 23.1 mm to (328.6, 167.2), turned to 3 degrees
- moved D4 22.9 mm to (101.5, 138.6), turned to 177 degrees
- moved SW5 22.4 mm to (101.0, 148.1), turned to -3 degrees
- moved SW1 21.3 mm to (82.0, 131.0), turned to -3 degrees
- moved SW4 21.2 mm to (102.0, 129.1), turned to -3 degrees
- moved SW2 20.4 mm to (81.0, 150.0), turned to -3 degrees
- moved SW9 19.6 mm to (120.9, 163.3), turned to -5 degrees
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Other:
- board outline added: 295.3 x 90.5 mm

Commit message: feat: 小指カラムをさげる part2
Parts:
- moved D1 4.29 mm to (81.5, 144.8)
- moved D2 4.29 mm to (80.5, 163.8)
- moved D3 4.29 mm to (79.5, 182.8)
- moved D37 4.29 mm to (327.1, 143.0)
- moved D38 4.29 mm to (328.1, 162.0)
- moved D39 4.29 mm to (329.1, 181.0)
- moved D4 4.29 mm to (101.5, 142.9)
- moved D40 4.29 mm to (347.5, 144.8)
- moved D41 4.29 mm to (349.5, 182.8)
- moved D5 4.29 mm to (100.5, 161.9)
- moved D6 4.29 mm to (99.5, 181.0)
- moved SW1 4.29 mm to (82.0, 135.3)
- moved SW2 4.29 mm to (81.0, 154.3)
- moved SW3 4.29 mm to (80.0, 173.3)
- moved SW37 4.29 mm to (326.6, 133.5)
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Other:
- outline, holes or cut-outs redrawn

Commit message: fix: 配線を修正
Connections:
- U1 pad 10: Row1 -> unconnected-(U1-GPIO7-Pad10)
- U1 pad 11: Row2 -> Col0
- U1 pad 12: Row3 -> Col1
- U1 pad 13: GND -> unconnected-(U1-GND-Pad13)
- U1 pad 14: Col0 -> Col2
- U1 pad 15: Col1 -> Col3
- U1 pad 16: Col2 -> Col4
- U1 pad 17: Col3 -> Col5
- U1 pad 18: GND -> unconnected-(U1-GND-Pad18)
- U1 pad 19: Col4 -> Row0
- U1 pad 20: Col5 -> Row1
- U1 pad 21: Col11 -> Row2
- U1 pad 22: Col10 -> Row3
- U1 pad 23: GND -> unconnected-(U1-GND-Pad23)
- U1 pad 24: Col9 -> Col6
- U1 pad 25: Col8 -> Col7
- U1 pad 26: Col7 -> Col8
- U1 pad 27: Col6 -> Col9
- U1 pad 28: GND -> unconnected-(U1-GND-Pad28)_0
- U1 pad 29: unconnected-(U1-GPIO22-Pad29) -> Col10
- U1 pad 3: GND -> unconnected-(U1-GND-Pad3)_0
- U1 pad 31: unconnected-(U1-GPIO26_ADC0-Pad31) -> Col11
- U1 pad 33: GND -> unconnected-(U1-AGND-Pad33)
- U1 pad 40: GND -> unconnected-(U1-VBUS-Pad40)_0
- U1 pad 8: GND -> unconnected-(U1-GND-Pad8)
- U1 pad 9: Row0 -> unconnected-(U1-GPIO6-Pad9)
