File: rev1/Assemble/first_keyboard.kicad_pcb (KiCad board)
At the start: 2 copper layers, 352.4 x 109.5 mm, 121 parts, among them SW1 SW_Push, SW10 SW_Push, SW11 SW_Push, SW12 SW_Push, SW13 SW_Push, SW14 SW_Push, SW15 SW_Push, SW16 SW_Push, SW17 SW_Push, SW18 SW_Push, SW19 SW_Push, SW2 SW_Push, SW20 SW_Push, SW21 SW_Push, SW22 SW_Push, SW23 SW_Push, SW24 SW_Push, SW25 SW_Push, SW26 SW_Push, SW27 SW_Push, SW28 SW_Push, SW29 SW_Push, SW3 SW_Push, SW30 SW_Push, SW31 SW_Push, SW32 SW_Push, SW33 SW_Push, SW34 SW_Push, SW35 SW_Push, SW36 SW_Push, SW37 SW_Push, SW38 SW_Push, SW39 SW_Push, SW4 SW_Push, SW40 SW_Push, SW41 SW_Push, SW42 SW_Push, SW43 SW_Push, SW44 SW_Push, SW45 SW_Push, SW46 SW_Push, SW47 SW_Push, SW48 SW_Push, SW49 SW_Push, SW5 SW_Push, SW50 SW_Push, SW51 SW_Push, SW52 SW_Push, SW53 SW_Push, SW54 SW_Push, SW55 SW_Push, SW56 SW_Push, SW57 SW_Push, SW58 SW_Push, SW59 SW_Push, SW6 SW_Push, SW60 SW_Push, SW7 SW_Push, SW8 SW_Push, SW9 SW_Push, U1 Pico

Commit message: feat: スペーサー穴追加
Parts:
- added Ref**: Val**, kbd_Hole:m2_Spacer_Hole_hex, F.Cu at (122.1, 76.8)
- added Ref**: Val**, kbd_Hole:m2_Spacer_Hole_hex, F.Cu at (122.1, 132.7)
- added Ref**: Val**, kbd_Hole:m2_Spacer_Hole_hex, F.Cu at (116.0, 147.0)
- added Ref**: Val**, kbd_Hole:m2_Spacer_Hole_hex, F.Cu at (294.8, 149.2)
- added Ref**: Val**, kbd_Hole:m2_Spacer_Hole_hex, F.Cu at (195.7, 130.2)
- added Ref**: Val**, kbd_Hole:m2_Spacer_Hole_hex, F.Cu at (218.6, 74.3)
- added Ref**: Val**, kbd_Hole:m2_Spacer_Hole_hex, F.Cu at (158.9, 75.6)
- added Ref**: Val**, kbd_Hole:m2_Spacer_Hole_hex, F.Cu at (78.6, 128.6)
- added Ref**: Val**, kbd_Hole:m2_Spacer_Hole_hex, F.Cu at (115.7, 52.7)
- added Ref**: Val**, kbd_Hole:m2_Spacer_Hole_hex, F.Cu at (291.0, 74.3)
- added Ref**: Val**, kbd_Hole:m2_Spacer_Hole_hex, F.Cu at (41.1, 52.7)
- added Ref**: Val**, kbd_Hole:m2_Spacer_Hole_hex, F.Cu at (387.5, 132.7)
- added Ref**: Val**, kbd_Hole:m2_Spacer_Hole_hex, F.Cu at (161.4, 130.2)
- added Ref**: Val**, kbd_Hole:m2_Spacer_Hole_hex, F.Cu at (214.8, 149.2)
- added Ref**: Val**, kbd_Hole:m2_Spacer_Hole_hex, F.Cu at (350.7, 75.6)
- added Ref**: Val**, kbd_Hole:m2_Spacer_Hole_hex, F.Cu at (387.5, 76.8)
- added Ref**: Val**, kbd_Hole:m2_Spacer_Hole_hex, F.Cu at (348.1, 130.2)
- added Ref**: Val**, kbd_Hole:m2_Spacer_Hole_hex, F.Cu at (41.1, 146.7)
- added Ref**: Val**, kbd_Hole:m2_Spacer_Hole_hex, F.Cu at (78.6, 71.4)
- added Ref**: Val**, kbd_Hole:m2_Spacer_Hole_hex, F.Cu at (313.8, 130.2)
Other:
- outline, holes or cut-outs redrawn

Commit message: feat: ネジ穴位置調整
Parts:
- removed Ref** (x20): Val**, kbd_Hole:m2_Spacer_Hole_hex
- added ref1: val, kbd_Hole:m2_Spacer_Hole_hex, F.Cu at (40.2, 52.7)
- added ref11: val, kbd_Hole:m2_Spacer_Hole_hex, F.Cu at (288.8, 73.0)
- added ref12: val, kbd_Hole:m2_Spacer_Hole_hex, F.Cu at (368.8, 76.8)
- added ref13: val, kbd_Hole:m2_Spacer_Hole_hex, F.Cu at (344.6, 131.4)
- added ref2: val, kbd_Hole:m2_Spacer_Hole_hex, F.Cu at (40.2, 146.7)
- added ref3: val, kbd_Hole:m2_Spacer_Hole_hex, F.Cu at (115.1, 52.7)
- added ref4: val, kbd_Hole:m2_Spacer_Hole_hex, F.Cu at (117.6, 131.4)
- added ref5: val, kbd_Hole:m2_Spacer_Hole_hex, F.Cu at (157.0, 75.6)
- added ref6: val, kbd_Hole:m2_Spacer_Hole_hex, F.Cu at (163.4, 131.4)
- added ref7: val, kbd_Hole:m2_Spacer_Hole_hex, F.Cu at (219.2, 73.0)
- added ref8: val, kbd_Hole:m2_Spacer_Hole_hex, F.Cu at (230.7, 154.3)
- added ref9: val, kbd_Hole:m2_Spacer_Hole_hex, F.Cu at (277.3, 154.3)
- moved U1 0.95 mm to (253.8, 97.6)
- moved D1 0.95 mm to (58.6, 66.7)
- moved D10 0.95 mm to (234.8, 90.5)
- moved D11 0.95 mm to (291.9, 90.5)
- moved D12 0.95 mm to (311.0, 85.7)
- moved D13 0.95 mm to (330.0, 85.7)
- moved D14 0.95 mm to (349.1, 90.5)
- moved D15 0.95 mm to (368.1, 90.5)
- moved D16 0.95 mm to (387.2, 90.5)
- moved D17 0.95 mm to (58.6, 85.7)
- moved D18 0.95 mm to (77.6, 85.7)
- moved D19 0.95 mm to (96.7, 85.7)
- moved D2 0.95 mm to (77.6, 66.7)
- moved D20 0.95 mm to (115.7, 85.7)
- moved D21 0.95 mm to (139.5, 109.5)
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Routing:
- net Net-(D17-K): track 0.00 -> 385.1 mm
- net Net-(D1-K): track 0.00 -> 379.4 mm
- net Net-(D33-K): track 0.00 -> 372.9 mm
- net Col0: track 0.00 -> 338.7 mm, vias 0 -> 1
- net Net-(D48-K): track 0.00 -> 285.8 mm
- net Col1: track 0.00 -> 272.9 mm, vias 0 -> 1
- net Col2: track 0.00 -> 255.2 mm, vias 0 -> 1
- net Col4: track 0.00 -> 250.6 mm
- net Col3: track 0.00 -> 204.2 mm, vias 0 -> 1
- net Col5: track 0.00 -> 171.8 mm
- net Col6: track 0.00 -> 166.6 mm, vias 0 -> 1
- net Col15: track 0.00 -> 162.6 mm
- net Col14: track 0.00 -> 146.2 mm
- net Col7: track 0.00 -> 145.7 mm, vias 0 -> 1
- net Col9: track 0.00 -> 142.9 mm
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