File: rev1/Assemble/first_keyboard.kicad_pcb (KiCad board)
At the start: 2 copper layers, 352.4 x 109.5 mm, 133 parts, among them SW1 SW_Push, SW10 SW_Push, SW11 SW_Push, SW12 SW_Push, SW13 SW_Push, SW14 SW_Push, SW15 SW_Push, SW16 SW_Push, SW17 SW_Push, SW18 SW_Push, SW19 SW_Push, SW2 SW_Push, SW20 SW_Push, SW21 SW_Push, SW22 SW_Push, SW23 SW_Push, SW24 SW_Push, SW25 SW_Push, SW26 SW_Push, SW27 SW_Push, SW28 SW_Push, SW29 SW_Push, SW3 SW_Push, SW30 SW_Push, SW31 SW_Push, SW32 SW_Push, SW33 SW_Push, SW34 SW_Push, SW35 SW_Push, SW36 SW_Push, SW37 SW_Push, SW38 SW_Push, SW39 SW_Push, SW4 SW_Push, SW40 SW_Push, SW41 SW_Push, SW42 SW_Push, SW43 SW_Push, SW44 SW_Push, SW45 SW_Push, SW46 SW_Push, SW47 SW_Push, SW48 SW_Push, SW49 SW_Push, SW5 SW_Push, SW50 SW_Push, SW51 SW_Push, SW52 SW_Push, SW53 SW_Push, SW54 SW_Push, SW55 SW_Push, SW56 SW_Push, SW57 SW_Push, SW58 SW_Push, SW59 SW_Push, SW6 SW_Push, SW60 SW_Push, SW7 SW_Push, SW8 SW_Push, SW9 SW_Push, U1 Pico

Commit message: update: madbd5 column
Connections:
- D1 pad 1: Net-(D1-K) -> Row0
- D10 pad 1: Net-(D1-K) -> Row0
- D11 pad 1: Net-(D1-K) -> Row0
- D12 pad 1: Net-(D1-K) -> Row0
- D13 pad 1: Net-(D1-K) -> Row0
- D14 pad 1: Net-(D1-K) -> Row0
- D15 pad 1: Net-(D1-K) -> Row0
- D16 pad 1: Net-(D1-K) -> Row0
- D17 pad 1: Net-(D17-K) -> Row1
- D18 pad 1: Net-(D17-K) -> Row1
- D19 pad 1: Net-(D17-K) -> Row1
- D2 pad 1: Net-(D1-K) -> Row0
- D20 pad 1: Net-(D17-K) -> Row1
- D21 pad 1: Net-(D17-K) -> Row1
- D22 pad 1: Net-(D17-K) -> Row1
- D23 pad 1: Net-(D17-K) -> Row1
- D24 pad 1: Net-(D17-K) -> Row1
- D25 pad 1: Net-(D17-K) -> Row1
- D26 pad 1: Net-(D17-K) -> Row1
- D27 pad 1: Net-(D17-K) -> Row1
- D28 pad 1: Net-(D17-K) -> Row1
- D29 pad 1: Net-(D17-K) -> Row1
- D3 pad 1: Net-(D1-K) -> Row0
- D30 pad 1: Net-(D17-K) -> Row1
- D31 pad 1: Net-(D17-K) -> Row1
- D32 pad 1: Net-(D17-K) -> Row1
- D33 pad 1: Net-(D33-K) -> Row2
- D34 pad 1: Net-(D33-K) -> Row2
- D35 pad 1: Net-(D33-K) -> Row2
- D36 pad 1: Net-(D33-K) -> Row2
- D37 pad 1: Net-(D33-K) -> Row2
- D38 pad 1: Net-(D33-K) -> Row2
- D39 pad 1: Net-(D33-K) -> Row2
- D4 pad 1: Net-(D1-K) -> Row0
- D40 pad 1: Net-(D33-K) -> Row2
- D41 pad 1: Net-(D33-K) -> Row2
- D42 pad 1: Net-(D33-K) -> Row2
- D43 pad 1: Net-(D33-K) -> Row2
- D44 pad 1: Net-(D33-K) -> Row2
- D45 pad 1: Net-(D33-K) -> Row2
- D46 pad 1: Net-(D33-K) -> Row2
- D47 pad 1: Net-(D33-K) -> Row2
- D48 pad 1: Net-(D48-K) -> Row3
- D49 pad 1: Net-(D48-K) -> Row3
- D5 pad 1: Net-(D1-K) -> Row0
- D50 pad 1: Net-(D48-K) -> Row3
- D51 pad 1: Net-(D48-K) -> Row3
- D52 pad 1: Net-(D48-K) -> Row3
- D53 pad 1: Net-(D48-K) -> Row3
- D54 pad 1: Net-(D48-K) -> Row3
- D55 pad 1: Net-(D48-K) -> Row3
- D56 pad 1: Net-(D48-K) -> Row3
- D57 pad 1: Net-(D48-K) -> Row3
- D58 pad 1: Net-(D58-K) -> Row4
- D59 pad 1: Net-(D58-K) -> Row4
- D6 pad 1: Net-(D1-K) -> Row0
- D60 pad 1: Net-(D58-K) -> Row4
- D7 pad 1: Net-(D1-K) -> Row0
- D8 pad 1: Net-(D1-K) -> Row0
- D9 pad 1: Net-(D1-K) -> Row0
- U1 pad 17: Col0 -> Row0
- U1 pad 19: Col0 -> Row1
- U1 pad 20: Col0 -> Row2
- U1 pad 21: Col0 -> Row3
- U1 pad 22: Col0 -> Row4
Routing:
- net Row1: track 0.00 -> 405.9 mm
- net Row0: track 0.00 -> 394.5 mm
- net Net-(D17-K): track 385.1 -> 0.00 mm
- net Row2: track 0.00 -> 381.2 mm
- net Net-(D1-K): track 379.4 -> 0.00 mm
- net Net-(D33-K): track 372.9 -> 0.00 mm
- net Row3: track 0.00 -> 319.2 mm
- net Net-(D48-K): track 285.8 -> 0.00 mm
- net Row4: track 0.00 -> 189.7 mm
- net Col0: track 338.7 -> 282.0 mm
- net Net-(D58-K): track 44.2 -> 0.00 mm
- net Col6: track 166.6 -> 196.6 mm, vias 1 -> 0
- net Col8: track 142.6 -> 166.6 mm, vias 1 -> 0
- net Col4: track 250.6 -> 229.8 mm
- net Col9: track 142.9 -> 133.8 mm
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