File: rev1/Assemble/first_keyboard.kicad_sch (KiCad schematic)
At the start: 121 parts, among them SW1 SW_Push, SW10 SW_Push, SW11 SW_Push, SW12 SW_Push, SW13 SW_Push, SW14 SW_Push, SW15 SW_Push, SW16 SW_Push, SW17 SW_Push, SW18 SW_Push, SW19 SW_Push, SW2 SW_Push, SW20 SW_Push, SW21 SW_Push, SW22 SW_Push, SW23 SW_Push, SW24 SW_Push, SW25 SW_Push, SW26 SW_Push, SW27 SW_Push, SW28 SW_Push, SW29 SW_Push, SW3 SW_Push, SW30 SW_Push, SW31 SW_Push, SW32 SW_Push, SW33 SW_Push, SW34 SW_Push, SW35 SW_Push, SW36 SW_Push, SW37 SW_Push, SW38 SW_Push, SW39 SW_Push, SW4 SW_Push, SW40 SW_Push, SW41 SW_Push, SW42 SW_Push, SW43 SW_Push, SW44 SW_Push, SW45 SW_Push, SW46 SW_Push, SW47 SW_Push, SW48 SW_Push, SW49 SW_Push, SW5 SW_Push, SW50 SW_Push, SW51 SW_Push, SW52 SW_Push, SW53 SW_Push, SW54 SW_Push, SW55 SW_Push, SW56 SW_Push, SW57 SW_Push, SW58 SW_Push, SW59 SW_Push, SW6 SW_Push, SW60 SW_Push, SW7 SW_Push, SW8 SW_Push, SW9 SW_Push, U1 Pico

Commit message: update: madbd5 column
Connections:
- net Col0: no longer U1.17 (GPIO13), U1.19 (GPIO14), U1.20 (GPIO15), U1.21 (GPIO16), U1.22 (GPIO17)
- net Row2: now reaches D33.1 (K), D34.1 (K), D35.1 (K), D36.1 (K), D37.1 (K), D38.1 (K), D39.1 (K), D40.1 (K), D41.1 (K), D42.1 (K), D43.1 (K), D44.1 (K), D45.1 (K), D46.1 (K), D47.1 (K)
- net Row2: now also U1.20 (GPIO15)
- net Row4: now reaches D58.1 (K), D59.1 (K), D60.1 (K)
- net Row4: now also U1.22 (GPIO17)
- net Row1: now reaches D17.1 (K), D18.1 (K), D19.1 (K), D20.1 (K), D21.1 (K), D22.1 (K), D23.1 (K), D24.1 (K), D25.1 (K), D26.1 (K), D27.1 (K), D28.1 (K), D29.1 (K), D30.1 (K), D31.1 (K), D32.1 (K)
- net Row1: now also U1.19 (GPIO14)
- net Row0: now reaches D1.1 (K), D10.1 (K), D11.1 (K), D12.1 (K), D13.1 (K), D14.1 (K), D15.1 (K), D16.1 (K), D2.1 (K), D3.1 (K), D4.1 (K), D5.1 (K), D6.1 (K), D7.1 (K), D8.1 (K), D9.1 (K)
- net Row0: now also U1.17 (GPIO13)
- net Row3: now reaches D48.1 (K), D49.1 (K), D50.1 (K), D51.1 (K), D52.1 (K), D53.1 (K), D54.1 (K), D55.1 (K), D56.1 (K), D57.1 (K)
- net Row3: now also U1.21 (GPIO16)
Changed lines of the file:
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@@
+	)
+	(junction
+		(at 162.56 236.22)
+		(diameter 0)
+		(color 0 0 0 0)
 	)
 	(junction
@@
 	)
 	(junction
+		(at 162.56 261.62)
+		(diameter 0)
+		(color 0 0 0 0)
+	)
+	(junction
 		(at 360.68 210.82)
 		(diameter 0)
@@
 	)
 	(junction
-		(at 152.4 279.4)
-		(diameter 0)
-		(color 0 0 0 0)
-	)
-	(junction
 		(at 334.01 177.8)
 		(diameter 0)
@@
 	)
 	(junction
+		(at 162.56 210.82)
+		(diameter 0)
+		(color 0 0 0 0)
+	)
+	(junction
 		(at 261.62 210.82)
 		(diameter 0)
@@
 	)
 	(junction
+		(at 162.56 287.02)
+		(diameter 0)
+		(color 0 0 0 0)
+	)
+	(junction
 		(at 234.95 228.6)
 		(diameter 0)
@@
 	(junction
 		(at 294.64 236.22)
+		(diameter 0)
+		(color 0 0 0 0)
+	)
+	(junction
+		(at 162.56 185.42)
 		(diameter 0)
 		(color 0 0 0 0)
@@
 	(wire
 		(pts
+			(xy 139.7 287.02) (xy 162.56 287.02)
+		)
+		(stroke
+			(width 0)
+			(type default)
+		)
+	)
+	(wire
+		(pts
 			(xy 344.17 210.82) (xy 360.68 210.82)
 		)
@@
 	(wire
 		(pts
-			(xy 139.7 228.6) (xy 152.4 228.6)
+			(xy 139.7 261.62) (xy 162.56 261.62)
 		)
 		(stroke
@@
 	(wire
 		(pts
-			(xy 139.7 177.8) (xy 152.4 177.8)
-		)
-		(stroke
-			(width 0)
-			(type default)
-		)
-	)
-	(wire
-		(pts
 			(xy 245.11 185.42) (xy 261.62 185.42)
 		)
@@
 	(wire
 		(pts
+			(xy 139.7 236.22) (xy 162.56 236.22)
+		)
+		(stroke
+			(width 0)
+			(type default)
+		)
+	)
+	(wire
+		(pts
 			(xy 251.46 228.6) (xy 251.46 254)
 		)
@@
 	(wire
 		(pts
-			(xy 139.7 203.2) (xy 152.4 203.2)
-		)
-		(stroke
-			(width 0)
-			(type default)
-		)
-	)
-	(wire
-		(pts
 			(xy 201.93 165.1) (xy 201.93 177.8)
 		)
@@
 	(wire
 		(pts
+			(xy 139.7 185.42) (xy 162.56 185.42)
+		)
+		(stroke
+			(width 0)
+			(type default)
+		)
+	)
+	(wire
+		(pts
 			(xy 179.07 261.62) (xy 195.58 261.62)
 		)
@@
 	(wire
 		(pts
+			(xy 139.7 210.82) (xy 162.56 210.82)
+		)
+		(stroke
+			(width 0)
+			(type default)
+		)
+	)
+	(wire
+		(pts
 			(xy 218.44 165.1) (xy 218.44 177.8)
 		)
@@
 	(wire
 		(pts
-			(xy 139.7 279.4) (xy 152.4 279.4)
-		)
-		(stroke
-			(width 0)
-			(type default)
-		)
-	)
-	(wire
-		(pts
 			(xy 400.05 165.1) (xy 400.05 177.8)
 		)
@@
 	(wire
 		(pts
-			(xy 139.7 254) (xy 152.4 254)
-		)
-		(stroke
-			(width 0)
-			(type default)
-		)
-	)
-	(wire
-		(pts
 			(xy 377.19 210.82) (xy 393.7 210.82)
 		)
@@
 	(global_label "Row2"
 		(shape input)
-		(at 139.7 228.6 180)
+		(at 139.7 236.22 180)
 		(fields_autoplaced yes)
 		(effects
@@
 		)
 		(property "Intersheetrefs" "${INTERSHEET_REFS}"
-			(at 131.7558 228.6 0)
+			(at 131.7558 236.22 0)
 			(effects
 				(font
@@
 	(global_label "Row4"
 		(shape input)
-		(at 139.7 279.4 180)
+		(at 139.7 287.02 180)
 		(fields_autoplaced yes)
 		(effects
@@
 		)
 		(property "Intersheetrefs" "${INTERSHEET_REFS}"
-			(at 131.7558 279.4 0)
+			(at 131.7558 287.02 0)
 			(effects
 				(font
@@
 	(global_label "Row3"
 		(shape input)
-		(at 139.7 254 180)
+		(at 139.7 261.62 180)
 		(fields_autoplaced yes)
 		(effects
@@
 		)
 		(property "Intersheetrefs" "${INTERSHEET_REFS}"
-			(at 131.7558 254 0)
+			(at 131.7558 261.62 0)
 			(effects
 				(font
@@
 	(global_label "Row1"
 		(shape input)
-		(at 139.7 203.2 180)
+		(at 139.7 210.82 180)
 		(fields_autoplaced yes)
 		(effects
@@
 		)
 		(property "Intersheetrefs" "${INTERSHEET_REFS}"
-			(at 131.7558 203.2 0)
+			(at 131.7558 210.82 0)
 			(effects
 				(font
@@
 	(global_label "Row0"
 		(shape input)
-		(at 139.7 177.8 180)
+		(at 139.7 185.42 180)
 		(fields_autoplaced yes)
 		(effects
@@
 		)
 		(property "Intersheetrefs" "${INTERSHEET_REFS}"
-			(at 131.7558 177.8 0)
-			(effects
-				(font
+			(at 131.7558 185.42 0)
+			(effects
+				(font
