File: rev1/Bottom/first_keyboard_bottom_top.kicad_pcb (KiCad board)
At the start: 2 copper layers, 352.4 x 109.5 mm, 12 parts

Commit message: remove: old gerber
Parts:
- moved ref7 1.37 mm to (219.2, 73.0)
- moved ref1 1.37 mm to (40.2, 52.7)
- moved ref2 1.37 mm to (40.2, 146.7)
- moved ref3 1.37 mm to (115.1, 52.7)
- moved ref5 1.37 mm to (157.0, 75.6)
- moved ref6 1.37 mm to (163.4, 131.4)
- moved ref8 1.37 mm to (230.7, 154.3)
- moved ref11 1.37 mm to (288.8, 73.0)
- moved ref4 1.37 mm to (117.6, 131.4)
- moved ref12 1.37 mm to (368.8, 76.8)
- moved ref13 1.37 mm to (344.6, 131.4)
- moved ref9 1.37 mm to (277.3, 154.3)
Other:
- outline, holes or cut-outs redrawn
